Commit message: limits

File: ex_2/urdf/bombel_dynamic.urdf (robot description, URDF)
Before this commit: robot Bombel1, 4 links, 3 joints
Joints:
- joint elbow: limit lower=0.0 upper=1.57 effort=1000.0 velocity=0.5 -> lower=0.0 upper=1 effort=1000.0 velocity=0.5; origin xyz=0.5 0 0 rpy=0 0 0 -> xyz=0.5 0 0 rpy=0 0 0.3
- joint shoulder: limit lower=-0.6 upper=-1.57 effort=1000.0 velocity=0.5 -> lower=0.3 upper=-0.3 effort=1000.0 velocity=0.5; origin xyz=0 0 0 rpy=-1.57 0 0 -> xyz=0 0 0 rpy=-1.57 -1 0
